Commit message: Adding final aidboat description and gazebo configurations

File: aidboat_description/urdf/aidboat_base.urdf.xacro (robot description, xacro)
@@ -5,5 +5,5 @@
 			<origin xyz="0.273998 ${reflect*(0.447)} -0.146" rpy="0 0 ${reflect*(-0.0244346)}"/>
 			<geometry>
-				<box size="2.002 0.286 0.292"/>
+				<box size="1.94 0.286 0.292"/>
 			</geometry>
 		</collision>
@@ -33,5 +33,5 @@
 			<origin rpy="0 0 0" xyz="0 0 0.292"/>
 			<geometry>
-				<mesh filename="package://aidboat_description/models/aidboat_base/mesh/AIDBOAT_Base.dae"/>
+				<mesh filename="package://aidboat_description/meshes/base/AIDBOAT_Base.dae"/>
 			</geometry>
 		</visual>

File: aidboat_gazebo/urdf/aidboat_gazebo.urdf.xacro (robot description, xacro)
@@ -1,11 +1,22 @@
 <?xml version="1.0"?>
-<!-- Basic WAM-V with gazebo plugins for dynamics -->
-<robot xmlns:xacro="http://ros.org/wiki/xacro"
-       name="aidboat">
-<xacro:arg name="thruster_namespace" default="thrusters/"/>
-<xacro:arg name="namespace" default="aidboat"/>
-<xacro:property name="thruster_namespace" value="$(arg thruster_namespace)" scope="global" />
-<xacro:property name="namespace" value="$(arg namespace)" scope="global" />
-<xacro:include filename="$(find aidboat_gazebo)/urdf/aidboat_gazebo.xacro"/>
-<xacro:aidboat_gazebo thruster_layout="$(find aidboat_gazebo)/urdf/thruster_layouts/aidboat_aft_thrusters.xacro"/>
+<robot xmlns:xacro="http://www.ros.org/wiki/xacro" name="aidboat">
+<!-- == Base vehicle == -->
+<xacro:include filename="$(find aidboat_description)/urdf/aidboat_base.urdf.xacro" />
+<!-- == Thrusters == -->
+<!--<xacro:include filename="$(find aidboat_gazebo)/urdf/thruster_layouts/thrusters.urdf" />-->
+<xacro:include filename="$(find aidboat_gazebo)/urdf/thrusters_gazebo.xacro" />
+<!-- == Hydrodynamics plugins == -->
+<xacro:include filename="$(find aidboat_gazebo)/urdf/aidboat_gazebo_dynamics_plugin.xacro" />
+<xacro:usv_dynamics_gazebo name="aidboat" />
+<!-- == Sensors == -->
+<xacro:include filename="$(find aidboat_gazebo)/urdf/sensors/camera.xacro" />
+<xacro:aidboat_camera name="camera" />
+<xacro:include filename="$(find aidboat_gazebo)/urdf/sensors/gps.xacro" />
+<xacro:aidboat_gps name="gps" />
+<xacro:include filename="$(find aidboat_gazebo)/urdf/sensors/imu.xacro" />
+<xacro:aidboat_imu name="imu" />
+<xacro:include filename="$(find aidboat_gazebo)/urdf/sensors/lidar2.xacro" />
+<xacro:aidboat_lidar name="lidar" />
+<xacro:include filename="$(find aidboat_gazebo)/urdf/sensors/p3d.xacro" />
+<xacro:p3d name="ground_truth_odometry" />
 </robot>

File: aidboat_gazebo/urdf/sensors/camera.xacro (robot description, xacro)
@@ -6,5 +6,5 @@
                 <origin xyz="0 -0.0147 -0.007" rpy="1.5708 0 1.5708"/>
                 <geometry>
-                    <mesh filename="package://aidboat_gazebo/models/camera/mesh/camera.dae"/>
+                    <mesh filename="package://aidboat_gazebo/meshes/camera.dae"/>
                 </geometry>
             </visual>
@@ -57,5 +57,5 @@
                     </noise>
                 </camera>
-                <plugin name="camera_plugin_${name}" filename="libgazebo_ros_camera.so">
+                <plugin name="aidboat_camera_plugin" filename="libgazebo_ros_camera.so">
                     <alwaysOn>true</alwaysOn>
                     <updateRate>0.0</updateRate>

File: aidboat_gazebo/urdf/sensors/gps.xacro (robot description, xacro)
@@ -1,5 +1,5 @@
 <?xml version="1.0" encoding="UTF-8"?>
 <robot xmlns:xacro="http://ros.org/wiki/xacro">
-    <xacro:macro name="aidboat_gps" params="name:=gps lat:=21.30996 lon:=-157.8901 elev:=0.0 update_rate:=20">
+    <xacro:macro name="aidboat_gps" params="name:=gps">
         <link name="${name}_link">
             <visual name="${name}_visual">
@@ -30,24 +30,21 @@
         </gazebo>
         <gazebo>
-            <plugin name="gps_plugin_${name}" filename="libhector_gazego_ros_gps.so">
-                <updateRate>${update_rate}</updateRate>
-                <alwaysOn>true</alwaysOn>
+            <plugin name="aidboat_gps_plugin" filename="libhector_gazebo_ros_gps.so">
+                <alwaysOn>1</alwaysOn>
+                <updateRate>15</updateRate>
                 <bodyName>${name}_link</bodyName>
-                <!-- Manually prepend namespace to tf frame -->
                 <frameId>aidboat/${name}_link</frameId>
-                <topicName>aidboat/sensors/gps/gps/fix</topicName>
-                <!-- Note that the hector_gazebo_ros_gps plugin uses NWU coordinates for reporting velocities. This may cause problems if localization requires velocity in ENU. See Issue #64 in VRX project for details. https://bitbucket.org/osrf/vrx/issues/64 -->
-                <velocityTopicName>aidboat/sensors/gps/gps/fix_velocity</velocityTopicName>
-                <!-- Location of origin of Gazebo Sand Island map -->
-                <referenceLatitude>${lat}</referenceLatitude>
-                <referenceLongitude>${lon}</referenceLongitude>
-                <referenceAltitude>${elev}</referenceAltitude>
-                <referenceHeading>90</referenceHeading>
-                <offset>0.0 0.0 0.0</offset>
+                <topicName>aidboat/sensors/gps/fix</topicName>
+                <velocityTopicName>aidboat/sensors/gps/velocity_fix</velocityTopicName>
+<!--                <referenceLatitude>21.30996</referenceLatitude>
+                <referenceLongitude>-157.8901</referenceLongitude>
+                <referenceAltitude>0</referenceAltitude>
+                <referenceHeading>90</referenceHeading>-->
+                <offset>0 0 0</offset>
                 <drift>0.0001 0.0001 0.0001</drift>
                 <gaussianNoise>0 0 0</gaussianNoise>
-                <velocityOffset>0.0 0.0 0.0</velocityOffset>
-                <velocityDrift>0.0 0.0 0.0</velocityDrift>
-                <velocityGaussianNoise>0.0 0.0 0.0</velocityGaussianNoise>
+                <velocityOffset>0 0 0</velocityOffset>
+                <velocityDrift>0 0 0</velocityDrift>
+                <velocityGaussianNoise>0 0 0</velocityGaussianNoise>
             </plugin>
         </gazebo>

File: aidboat_gazebo/urdf/sensors/imu.xacro (robot description, xacro)
@@ -1,5 +1,5 @@
 <?xml version="1.0"?>
 <robot xmlns:xacro="http://ros.org/wiki/xacro">
-    <xacro:macro name="aidboat_imu" params="name:=imu update_rate:=50">
+    <xacro:macro name="aidboat_imu" params="name:=imu">
         <link name="${name}_link">
             <visual name="${name}_visual">
@@ -30,8 +30,8 @@
         </gazebo>
         <gazebo>
-            <plugin name="imu_plugin_${name}" filename="libhector_gazebo_ros_imu.so">
-                <updateRate>${update_rate}</updateRate>
+            <plugin name="aidboat_imu_plugin" filename="libhector_gazebo_ros_imu.so">
+                <updateRate>50</updateRate>
                 <bodyName>${name}_link</bodyName>
-                <topicName>aidboat/sensors/imu/imu/data</topicName>
+                <topicName>aidboat/sensors/imu/data</topicName>
                 <serviceName>aidboat/sensors/imu_service</serviceName>
                 <!--Manually prepend namespace to tf frame -->

File: aidboat_gazebo/urdf/sensors/lidar2.xacro (robot description, xacro)
@@ -6,5 +6,5 @@
                 <origin xyz="0 0 0" rpy="0 0 -1.5708"/>
                 <geometry>
-                    <mesh filename="package://aidboat_description/meshes/lidar.stl"/>
+                    <mesh filename="package://aidboat_gazebo/meshes/lidar.stl"/>
                     <!--<cylinder radius="0.0525" length="0.152"/>-->
                 </geometry>
@@ -33,14 +33,12 @@
             <child link="${name}_laser" />
         </joint>
-        <gazebo reference="${name}_link">
-            <mu1>0.2</mu1>
-            <mu2>0.2</mu2>
-        </gazebo>
-        <gazebo reference="${name}_link">
-            <sensor type="lidar" name="${name}_sensor">
-                <always_on>true</always_on>
+        <material name="black">
+            <color rgba="0 0 0 1.0"/>
+        </material>
+        <gazebo reference="${name}_laser">
+            <sensor type="ray" name="${name}_sensor">
+                <pose>0 0 0 0 0 0</pose>
+                <visualize>False</visualize>
                 <update_rate>15</update_rate>
-                <pose>0 0 0 0 0 0</pose>
-                <visualize>false</visualize>
                 <ray>
                     <scan>
@@ -57,11 +55,13 @@
                         <resolution>0.01</resolution>
                     </range>
+                    <noise>
+                        <type>gaussian</type>
+                        <mean>0.0</mean>
+                        <stddev>0.01</stddev>
+                    </noise>
                 </ray>
-                <plugin name="lidar_plugin_${name}" filename="libgazebo_ros_laser.so">
-                    <gaussianNoise>0.005</gaussianNoise>
-                    <alwaysOn>true</alwaysOn>
-                    <updateRate>15</updateRate>
-                    <topicName>/aidboat/laser/scan</topicName>
-                    <frameName>${name}_link</frameName>
+                <plugin name="aidboat_${name}_plugin" filename="libgazebo_ros_laser.so">
+                    <topicName>/aidboat/sensors/laser/scan</topicName>
+                    <frameName>${name}_laser</frameName>
                 </plugin>
             </sensor>

File: aidboat_gazebo/urdf/sensors/p3d.xacro (robot description, xacro)
@@ -3,5 +3,5 @@
   <xacro:macro name="p3d" params="name:=ground_truth_odometry">
     <gazebo>
-      <plugin name="p3d_plugin_${name}" filename="libgazebo_ros_p3d.so">
+      <plugin name="aidboat_p3d_plugin" filename="libgazebo_ros_p3d.so">
         <bodyName>base_link</bodyName>
         <frameName>map</frameName>

File: aidboat_gazebo/urdf/thrusters_gazebo.xacro (robot description, xacro)
@@ -1,88 +1,27 @@
 <?xml version="1.0"?>
 <robot xmlns:xacro="http://ros.org/wiki/xacro" name="aidboat-thrusters">
-  <!-- Macro for inserting an engine with its propeller. -->
-  <xacro:macro name="engine" params="prefix reflect reflect2">
-    <link name="${prefix}_engine_link">
-      <visual>
-        <origin xyz="0 0 0" rpy="0 0 ${reflect*(0.0244346)}" />
-        <geometry>
-          <mesh filename="package://aidboat_description/models/engine/mesh/${prefix}_engine.dae"/>
-        </geometry>
-      </visual>
-      <collision>
-        <origin xyz="0.011 0 0" rpy="0 1.5708 ${reflect*(0.0244346)}" />
-        <geometry>
-          <cylinder length="0.113" radius="0.05" />
-        </geometry>
-      </collision>
-      <inertial>
-        <mass value="0.126"/>
-        <inertia ixx="0.00002900992" ixy="0" ixz="0" iyy="0.00002900992" iyz="0" izz="0.0001575"/>
-      </inertial>
-    </link>
-    <link name="${prefix}_propeller_link">
-      <visual>
-        <origin xyz="0 0 0" rpy="0 0 ${reflect*(0.0244346)}" />
-        <geometry>
-          <mesh filename="package://aidboat_description/models/propeller/mesh/${prefix}_propeller.dae" />
-        </geometry>
-      </visual>
-      <collision>
-        <origin xyz="0.011 0 0" rpy="0 1.5708 ${reflect*(0.0244346)}" />
-        <geometry>
-          <cylinder length="0.03" radius="0.0381" />
-        </geometry>
-      </collision>
-      <inertial>
-        <mass value="0.030"/>
-        <inertia ixx="0.00000058378" ixy="0" ixz="0" iyy="0.00000058378" iyz="0" izz="0.00002177415" />
-      </inertial>
-    </link>
-    <joint name="${prefix}_chasis_engine_joint" type="revolute">
-      <axis xyz="1 0 0"/>
-      <limit lower="0" upper="0" effort="0" velocity="0"/>
-      <origin xyz="-0.741 ${reflect2*(0.47)} -0.016" rpy="0 0 0"/>
-      <parent link="base_link"/>
-      <child link="${prefix}_engine_link"/>
-    </joint>
-    <joint name="${prefix}_engine_propeller_joint" type="continuous">
-      <axis rpy="0 0 0" xyz="1 0 0" />
-      <parent link="${prefix}_engine_link"/>
-      <child link="${prefix}_propeller_link"/>
-      <origin xyz="0 0 0" rpy="0 0 0"/>
-      <limit effort="0.7250" velocity="369.97489" />
-      <dynamics friction="0.05" damping="0.05" />
-    </joint>
-    <gazebo reference="${prefix}_engine_link">
-      <mu1>0.2</mu1>
-      <mu2>0.2</mu2>
-    </gazebo>
-    <gazebo reference="${prefix}_propeller_link">
-      <mu1>0.2</mu1>
-      <mu2>0.2</mu2>
-    </gazebo>
-  </xacro:macro>
+  <xacro:include filename="$(find aidboat_description)/urdf/thrusters.xacro" />
+  <xacro:thrusters prefix="right" reflect="1" reflect2="-1"/>
+  <xacro:thrusters prefix="left" reflect="-1" reflect2="1"/>
   <gazebo>
-    <plugin name="aidboat_gazebo_thrust" filename="libusv_gazebo_thrust_plugin.so" xmlns:xacro="http://ros.org/wiki/xacro">
-      <cmdTimeout>1.0</cmdTimeout>
-      <thruster>
-        <linkName>left_propeller_link</linkName>
-        <propJointName>left_engine_propeller_joint</propJointName>
-        <engineJointName>left_chasis_engine_joint</engineJointName>
-        <cmdTopic>left_thrust_cmd</cmdTopic>
-        <angleTopic>left_thrust_angle</angleTopic>
-        <enableAngle>false</enableAngle>
-      </thruster>
-      <thruster>
-        <linkName>right_propeller_link</linkName>
-        <propJointName>right_engine_propeller_joint</propJointName>
-        <engineJointName>right_chasis_engine_joint</engineJointName>
-        <cmdTopic>right_thrust_cmd</cmdTopic>
-        <angleTopic>right_thrust_angle</angleTopic>
-        <enableAngle>false</enableAngle>
-      </thruster>
-    </plugin>
+    <xacro:macro name="thrusters_plugin" params="prefix">
+      <plugin name="aidboat_gazebo_thrust" filename="libusv_gazebo_thrust_plugin.so" xmlns:xacro="http://ros.org/wiki/xacro">
+        <cmdTimeout>1.0</cmdTimeout>
+        <thruster>
+          <linkName>${prefix}_propeller_link</linkName>
+          <propJointName>${prefix}_engine_propeller_joint</propJointName>
+          <engineJointName>${prefix}_chasis_engine_joint</engineJointName>
+          <cmdTopic>${prefix}_thrust_cmd</cmdTopic>
+          <angleTopic>${prefix}_thrust_angle</angleTopic>
+          <enableAngle>false</enableAngle>
+          <mappingType>0</mappingType>
+          <maxCmd>1.0</maxCmd>
+          <maxForceFwd>51.4849</maxForceFwd>
+          <maxForceRev>-40.2073</maxForceRev>
+        </thruster>
+      </plugin>
+    </xacro:macro>
+    <xacro:thrusters_plugin prefix="right"/>
+    <xacro:thrusters_plugin prefix="left"/>
   </gazebo>
-<xacro:engine prefix="right" reflect="1" reflect2="-1"/>
-<xacro:engine prefix="left" reflect="-1" reflect2="1"/>
 </robot>

Commit message: completed description package and start of navigation

File: aidboat_description/urdf/aidboat_base.urdf.xacro (robot description, xacro)
@@ -3,5 +3,5 @@
 	<xacro:macro name="collisions" params="prefix reflect">
 		<collision name="${prefix}_hull">
-			<origin xyz="0.273998 ${reflect*(0.447)} -0.146" rpy="0 0 ${reflect*(-0.0244346)}"/>
+			<origin xyz="0.273998 ${reflect*(0.447)} 0.146" rpy="0 0 ${reflect*(-0.0244346)}"/>
 			<geometry>
 				<box size="1.94 0.286 0.292"/>
@@ -23,5 +23,5 @@
 		</inertial>
 		<collision name="top_base">
-			<origin xyz="0 0 0.1255" rpy="0 0 0"/>
+			<origin xyz="0 0 0.418" rpy="0 0 0"/>
 			<geometry>
 				<box size="0.73 1.15767 0.251"/>

File: aidboat_gazebo/urdf/aidboat_gazebo.urdf.xacro (robot description, xacro)
@@ -4,5 +4,4 @@
 <xacro:include filename="$(find aidboat_description)/urdf/aidboat_base.urdf.xacro" />
 <!-- == Thrusters == -->
-<!--<xacro:include filename="$(find aidboat_gazebo)/urdf/thruster_layouts/thrusters.urdf" />-->
 <xacro:include filename="$(find aidboat_gazebo)/urdf/thrusters_gazebo.xacro" />
 <!-- == Hydrodynamics plugins == -->

File: aidboat_gazebo/urdf/sensors/gps.xacro (robot description, xacro)
@@ -31,16 +31,16 @@
         <gazebo>
             <plugin name="aidboat_gps_plugin" filename="libhector_gazebo_ros_gps.so">
-                <alwaysOn>1</alwaysOn>
+                <alwaysOn>true</alwaysOn>
                 <updateRate>15</updateRate>
                 <bodyName>${name}_link</bodyName>
-                <frameId>aidboat/${name}_link</frameId>
+                <frameId>${name}_link</frameId>
                 <topicName>aidboat/sensors/gps/fix</topicName>
-                <velocityTopicName>aidboat/sensors/gps/velocity_fix</velocityTopicName>
-<!--                <referenceLatitude>21.30996</referenceLatitude>
+                <velocityTopicName>aidboat/sensors/gps/fix_velocity</velocityTopicName>
+                <referenceLatitude>21.30996</referenceLatitude>
                 <referenceLongitude>-157.8901</referenceLongitude>
                 <referenceAltitude>0</referenceAltitude>
-                <referenceHeading>90</referenceHeading>-->
+                <referenceHeading>90</referenceHeading>
                 <offset>0 0 0</offset>
-                <drift>0.0001 0.0001 0.0001</drift>
+                <drift>0 0 0</drift>
                 <gaussianNoise>0 0 0</gaussianNoise>
                 <velocityOffset>0 0 0</velocityOffset>

File: aidboat_gazebo/urdf/sensors/imu.xacro (robot description, xacro)
@@ -36,5 +36,5 @@
                 <serviceName>aidboat/sensors/imu_service</serviceName>
                 <!--Manually prepend namespace to tf frame -->
-                <frameId>aidboat/${name}_link</frameId>
+                <frameId>${name}_link</frameId>
                 <alwaysOn>true</alwaysOn>
                 <accelOffset>0.0 0.0 0.0</accelOffset>

Commit message: changes inertia matrix

File: aidboat_description/urdf/aidboat_base.urdf.xacro (robot description, xacro)
@@ -20,5 +20,5 @@
 			<mass value="32.712"/>
 			<origin xyz="0 0.26377 0.02064" rpy="0 0 0"/>
-			<inertia ixx="4.662514672" ixy="0" ixz="0" iyy="12.57628507" iyz="0" izz="15.22053986"/>
+			<inertia ixx="4.4927206" ixy="0" ixz="0" iyy="11.783203" iyz="0" izz="14.626694"/>
 		</inertial>
 		<collision name="top_base">
